Commit message: A simple test script file has been created which creates a .xml file from a .xacro file with given params. The next step is to figure out which parts of gate.xacro need to be abstracted out, and what range their values should be. We should look into creating a script to generate sequences of parms which we can then use to automate test parameter creation

File: src/simulator/scenes/gate/gate.xacro (robot description, xacro)
@@ -2,5 +2,21 @@
 <!DOCTYPE UWSimScene SYSTEM "UWSimScene.dtd" >
 <UWSimScene xmlns:xacro="http://www.ros.org/wiki/xacro">
-<xacro:property name="the_yaw" value="-0.75" />
+<!-- args -->
+<xacro:arg name="test#" default="0"/>
+<xacro:arg name="roll" default="0"/>
+<xacro:arg name="pitch" default="0"/>
+<xacro:arg name="yaw" default="0.75"/>
+<xacro:arg name="xpos" default="0"/>
+<xacro:arg name="ypos" default="3.5"/>
+<xacro:arg name="zpos" default="1.5"/>
+<!-- arg values -->
+<xacro:property name="roll_val" value="$(arg roll)"/>
+<xacro:property name="pitch_val" value="$(arg pitch)"/>
+<xacro:property name="yaw_val" value="$(arg yaw)"/>
+<xacro:property name="xpos_val" value="$(arg xpos)"/>
+<xacro:property name="ypos_val" value="$(arg ypos)"/>
+<xacro:property name="zpos_val" value="$(arg zpos)"/>
+<!--To run with yaw param, run "rosrun xacro xacro %%inorder gate.xacro > ./gate.xml yaw:=**enter param here**">-->
+<!-- NOTE: because you cannot have a dash in xml comments, replace each % with a dash-->
   <oceanState>
     <windx> 0.04 </windx>
@@ -70,5 +86,5 @@
     </lookAt>
   </camera>
-  <!--Start of Vehicle parameters-->
+  <!--start of vehicle parameters-->
   <vehicle>
     <name>girona500</name>
@@ -82,13 +98,12 @@
     </jointValues>
     <position>
-      <x> 0</x>
-      <y> 3.5 </y>
-      <z> 1.5 </z>
-    </position>
-    <orientation>
-      <r>0</r>
-      <p>0</p>
-      <!-- <y>-0.75</y> -->
-      <y>${the_yaw}</y>
+      <x>${xpos_val}</x>
+      <y>${ypos_val}</y>
+      <z>${zpos_val}</z>
+    </position>
+    <orientation>
+      <r>${roll_val}</r>
+      <p>${pitch_val}</p>
+      <y>${yaw_val}</y>
     </orientation>
     <virtualCamera>
