Commit message: Added pysimtest library, needs testing

File: src/simulator/testing/run/scenes/gate/gate.xacro (robot description, xacro)
@@ -1,12 +1,21 @@
-<?xml version="1.0" ?>
-<!-- =================================================================================== -->
-<!-- |    This document was autogenerated by xacro from /home/owen/Documents/Subbots/Jormungandr/src/simulator/simtest/run/scenes/gate/gate.xacro | -->
-<!-- |    EDITING THIS FILE BY HAND IS NOT RECOMMENDED                                 | -->
-<!-- =================================================================================== -->
-<!DOCTYPE UWSimScene
-  SYSTEM 'UWSimScene.dtd'>
+<?xml version="1.0"?>
+<!DOCTYPE UWSimScene SYSTEM "UWSimScene.dtd" >
 <UWSimScene xmlns:xacro="http://www.ros.org/wiki/xacro">
-  <!--To run with yaw param, run "rosrun xacro xacro %%inorder gate.xacro > ./gate.xml yaw:=**enter param here**">-->
-  <!-- NOTE: because you cannot have a dash in xml comments, replace each % with a dash-->
+<!-- args -->
+<xacro:arg name="vehicle_x_pos" default="0"/>
+<xacro:arg name="vehicle_y_pos" default="3.5"/>
+<xacro:arg name="vehicle_z_pos" default="1.5"/>
+<xacro:arg name="vehicle_r_rot" default="0"/>
+<xacro:arg name="vehicle_p_rot" default="0"/>
+<xacro:arg name="vehicle_y_rot" default="0.75"/>
+<!-- arg values -->
+<xacro:property name="vehicle_x_pos_val" value="$(arg vehicle_x_pos)"/>
+<xacro:property name="vehicle_y_pos_val" value="$(arg vehicle_y_pos)"/>
+<xacro:property name="vehicle_z_pos_val" value="$(arg vehicle_z_pos)"/>
+<xacro:property name="vehicle_r_rot_val" value="$(arg vehicle_r_rot)"/>
+<xacro:property name="vehicle_p_rot_val" value="$(arg vehicle_p_rot)"/>
+<xacro:property name="vehicle_y_rot_val" value="$(arg vehicle_y_rot)"/>
+<!--To run with yaw param, run "rosrun xacro xacro %%inorder gate.xacro > ./gate.xml yaw:=**enter param here**">-->
+<!-- NOTE: because you cannot have a dash in xml comments, replace each % with a dash-->
   <oceanState>
     <windx> 0.04 </windx>
@@ -23,7 +32,7 @@
       <density> 0.1</density>
       <color>
-        <r>0</r>
-        <g>0.05</g>
-        <b>0.3</b>
+	<r>0</r>
+	<g>0.05</g>
+	<b>0.3</b>
       </color>
     </fog>
@@ -88,12 +97,12 @@
     </jointValues>
     <position>
-      <x>2</x>
-      <y>3</y>
-      <z>4</z>
-    </position>
-    <orientation>
-      <r>4</r>
-      <p>5</p>
-      <y>6</y>
+      <x>${vehicle_x_pos_val}</x>
+      <y>${vehicle_y_pos_val}</y>
+      <z>${vehicle_z_pos_val}</z>
+    </position>
+    <orientation>
+      <r>${vehicle_r_rot_val}</r>
+      <p>${vehicle_p_rot_val}</p>
+      <y>${vehicle_y_rot_val}</y>
     </orientation>
     <virtualCamera>
@@ -510,10 +519,10 @@
     </WorldToROSTF>
     <ArmToROSJointState>
-      <topic>/uwsim/joint_state</topic>
-      <vehicleName> girona500 </vehicleName>
+	<topic>/uwsim/joint_state</topic>
+	<vehicleName> girona500 </vehicleName>
     </ArmToROSJointState>
     <ROSJointStateToArm>
-      <topic>/uwsim/joint_state_command</topic>
-      <vehicleName> girona500 </vehicleName>
+	<topic>/uwsim/joint_state_command</topic>
+	<vehicleName> girona500 </vehicleName>
     </ROSJointStateToArm>
     <VirtualCameraToROSImage>
